File: Porta logica/$Porta logica.sch (KiCad schematic (older format))
At the start: 56 parts, among them P1 Input, P2 Out, SW1 SW_PUSH, SW2 SW_PUSH, U1 74HC595, U2 74HC595, U3 74HC00, U4 74HC595

Commit message: correzione bug, migliorie grafiche
Parts:
- removed unit 1 of U3
Changed lines of the file:
@@
 F1 "clock.sch" 50
 F2 "Clk" O R 8600 5950 60
-F3 "Reset" O R 8600 6200 60
+F3 "~Reset" O R 8600 6200 60
 $EndSheet
-$Comp
-L 74HC00 U3
-U 1 1 555C716A
-P 9600 6600
-F 0 "U3" H 9600 6650 60  0000 C CNN
-F 1 "74HC00" H 9600 6500 60  0000 C CNN
-F 2 "~" H 9600 6600 60  0000 C CNN
-F 3 "~" H 9600 6600 60  0000 C CNN
-	1    9600 6600
-	1    0    0    -1
-$EndComp
 $Comp
 L CONN_2 P2
@@
 Wire Wire Line
 	750  1600 750  1800
-Connection ~ 9000 6600
 Wire Wire Line
 	8700 6200 8600 6200
 Wire Wire Line
-	8700 6600 8700 6200
-Wire Wire Line
-	9000 6600 8700 6600
-Wire Wire Line
-	9000 6500 9000 6700
-Wire Wire Line
-	1500 1800 2050 1800
+	8700 6450 8700 6200
+Wire Wire Line
+	1500 1800 1600 1800
+Wire Wire Line
+	1600 1800 2050 1800
 Wire Wire Line
 	7400 6250 7250 6250
@@
 Connection ~ 5100 1500
 Wire Wire Line
-	9800 3250 9800 4250
+	9800 3250 9800 3550
+Wire Wire Line
+	9800 3550 9800 3850
+Wire Wire Line
+	9800 3850 9800 4150
+Wire Wire Line
+	9800 4150 9800 4250
 Wire Wire Line
 	8250 4150 8750 4150
@@
 Connection ~ 7650 2000
 Wire Wire Line
-	7650 1900 7650 2100
+	7650 1900 7650 2000
+Wire Wire Line
+	7650 2000 7650 2100
 Wire Wire Line
 	7500 2000 7650 2000
@@
 Connection ~ 1600 5400
 Wire Wire Line
-	1500 5400 2100 5400
+	1500 5400 1600 5400
+Wire Wire Line
+	1600 5400 2100 5400
 Connection ~ 1600 1800
 Wire Wire Line
@@
 	1600 5950 1600 6050
 Wire Wire Line
-	1600 4000 1600 5450
+	1600 4000 1600 5400
+Wire Wire Line
+	1600 5400 1600 5450
 Wire Wire Line
 	750  5400 900  5400
@@
 	2050 6100 2050 6000
 Wire Wire Line
-	9000 5850 9000 6050
+	9000 5850 9000 5950
+Wire Wire Line
+	9000 5950 9000 6050
 Wire Wire Line
 	2050 2300 1800 2300
@@
 	3500 5400 3500 4800
 Wire Wire Line
-	5150 4800 5150 7050
+	5150 4800 5150 5100
+Wire Wire Line
+	5150 5100 5150 5400
+Wire Wire Line
+	5150 5400 5150 5700
+Wire Wire Line
+	5150 5700 5150 6000
+Wire Wire Line
+	5150 6000 5150 6300
+Wire Wire Line
+	5150 6300 5150 6600
+Wire Wire Line
+	5150 6600 5150 6900
+Wire Wire Line
+	5150 6900 5150 7050
 Wire Wire Line
 	4650 4800 4500 4800
@@
 	3450 1800 3450 1200
 Wire Wire Line
-	5100 1200 5100 3450
+	5100 1200 5100 1500
+Wire Wire Line
+	5100 1500 5100 1800
+Wire Wire Line
+	5100 1800 5100 2100
+Wire Wire Line
+	5100 2100 5100 2400
+Wire Wire Line
+	5100 2400 5100 2700
+Wire Wire Line
+	5100 2700 5100 3000
+Wire Wire Line
+	5100 3000 5100 3300
+Wire Wire Line
+	5100 3300 5100 3450
 Wire Wire Line
 	4600 1200 4450 1200
@@
 Wire Wire Line
 	1850 5700 2100 5700
-Text Label 10500 6600 2    60   ~ 0
+Text Label 9150 6450 2    60   ~ 0
 reset
-Wire Wire Line
-	10200 6600 10500 6600
 Text Label 3700 3300 0    60   ~ 0
 in_a
@@
 	1650 1500 1600 1500
 Wire Wire Line
-	1600 1500 1600 3800
+	1600 1500 1600 1800
+Wire Wire Line
+	1600 1800 1600 3800
 Wire Wire Line
 	1600 3800 1050 3800
@@
 F3 "Vcc" O R 7250 6000 60
 $EndSheet
+Wire Wire Line
+	8700 6450 9150 6450
+Wire Wire Line
+	9150 6450 9150 6450
 $EndSCHEMATC
