File: Porta logica/$clock.sch (KiCad schematic (older format))
At the start: 14 parts, among them P4 Clock, U6 74HC00, U7 LM555N

Commit message: correzione bug, migliorie grafiche
Parts:
- added R?: 10k, ~, symbol R
- gave numbers to parts that had none: 1
Connections:
- net Clk: now also R?.1
- net GND: now also C3.2, R?.2; no longer R26.2, R28.2, R29.2
- net VCC: now also R26.1, R28.1, R29.1; no longer C3.1
- net at P4.2 (PM), U6.1, U6.4: now also R26.2; no longer R26.1
- removed net Reset: C3.2, R28.1, R29.1, U6.13
- new net ~Reset: C3.1, R28.2, R29.2, U6.13
- no-connect marks 0 -> 1
Other:
- moved on the sheet: C3, R26, R28, R29
